File: medidor-2.sch (EAGLE design)
At the start: 30 parts

Commit message: ahora si funciona
Parts:
- removed J4: (no value), SparkFun-Connectors:CONN_063.5MM-6
- added J1, J2: (no value), SparkFun-Connectors:CONN_03-SCREW-5MM
Connections:
- net 1-A: now also 4511-2.7; no longer 4511-1.7
- net 1-B: now also 4511-2.1; no longer 4511-1.1
- net 1-C: now also 4511-2.2; no longer 4511-1.2
- net 1-D: now also 4511-2.6; no longer 4511-1.6
- net 2-A: now also 4511-1.7; no longer 4511-2.7
- net 2-B: now also 4511-1.1; no longer 4511-2.1
- net 2-C: now also 4511-1.2; no longer 4511-2.2
- net 2-D: now also 4511-1.6, J1.2; no longer 4511-2.6, J4.2
- net 5V: now also J2.3; no longer J4.6
- net CLOCK-EXT: now also J2.2; no longer J4.5
- net ENABLE-A: now also J2.1; no longer J4.4
- net GND: now also J1.1; no longer J4.1
- net RESET-A-B: now also J1.3; no longer J4.3
