File: medidor-2.brd (EAGLE design)
At the start: 30 parts

Commit message: ahora si funciona
Parts:
- removed J4: (no value), SparkFun-Connectors:SCREWTERMINAL-3.5MM-6
- added J1, J2: (no value), SparkFun-Connectors:SCREWTERMINAL-5MM-3
- moved D1 9.25 mm to (105.4, 11.4)
- moved C1 1.27 mm to (40.6, 44.5)
- turned 4518 to 90 degrees
Connections:
- net 1-A: now also 4511-2.7; no longer 4511-1.7
- net 1-B: now also 4511-2.1; no longer 4511-1.1
- net 1-C: now also 4511-2.2; no longer 4511-1.2
- net 1-D: now also 4511-2.6; no longer 4511-1.6
- net 2-A: now also 4511-1.7; no longer 4511-2.7
- net 2-B: now also 4511-1.1; no longer 4511-2.1
- net 2-C: now also 4511-1.2; no longer 4511-2.2
- net 2-D: now also 4511-1.6, J1.2; no longer 4511-2.6, J4.2
- net 5V: now also J2.3; no longer J4.6
- net CLOCK-EXT: now also J2.2; no longer J4.5
- net ENABLE-A: now also J2.1; no longer J4.4
- net GND: now also J1.1; no longer J4.1
- net RESET-A-B: now also J1.3; no longer J4.3
Routing:
- net 1-D: track 101.4 -> 52.9 mm, vias 4 -> 2
- net 1-C: track 69.2 -> 30.5 mm
- net RESET-A-B: track 160.8 -> 187.8 mm
- net 2-A: track 47.5 -> 24.2 mm, vias 0 -> 2
- net 1-A: track 24.2 -> 44.5 mm, vias 2 -> 0
- net 1-B: track 48.1 -> 30.5 mm
- net 2-C: track 30.5 -> 45.7 mm
- net D1-A: track 49.8 -> 34.6 mm, vias 2 -> 1
- net 2-D: track 104.4 -> 89.7 mm, vias 2 -> 3
- net 2-B: track 30.5 -> 45.0 mm
- net D2-A: track 49.2 -> 35.9 mm, vias 2 -> 1
- net CLOCK-A: track 48.4 -> 40.0 mm
- net CLOCK-EXT: track 46.8 -> 50.1 mm
- net ENABLE-A: track 91.4 -> 93.8 mm
- net GND: track 369.5 -> 371.3 mm, vias 0 -> 3
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
Commit message: flatcam
Parts:
- moved 4511-2 25.4 mm to (82.5, 63.5)
- moved 4518 25.4 mm to (54.6, 45.7)
- moved J2 25.4 mm to (59.7, 10.2)
- moved R1 25.4 mm to (72.4, 33.0)
- moved R11 25.4 mm to (91.4, 78.7)
- moved R4 25.4 mm to (91.4, 34.3)
- moved R5 25.4 mm to (73.7, 78.7)
- moved R7 25.4 mm to (78.7, 78.7)
- moved R8 25.4 mm to (81.3, 78.7)
- moved R9 25.4 mm to (83.8, 78.7)
- moved S1 25.4 mm to (91.4, 24.1)
- moved R16 25.4 mm to (27.9, 77.5)
- moved R2 25.4 mm to (30.5, 34.3)
- moved 4511-1 25.4 mm to (26.7, 63.5)
- moved 555 25.4 mm to (17.8, 33.0)
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